File: devkit/ZSWatch-Watch-DevKit.kicad_pcb (KiCad board)
At the start: 4 copper layers, 100 x 70 mm, 125 parts, among them IC401 nPM1300-QEXX, IC501 APDS-9306-065, IC502 BMI270, IC503 LIS2MDLTR, IC504 BMP581, IC505 DRV2603RUNT, IC506 PCA9306JK, IC507 RV-8263-C8, IC601 FAN5622SX, IC602 USBLC6-2P6, IC603 MX25U51245GZ4I00, IC604 NTS0104GU12, M601 NORA-B106, Q401 PMZ550UNEYL, Q402 PMZ550UNEYL, Q403 PMZ550UNEYL, Q404 PMZB320UPEYL, X401 Battery, X402 Battery, X403 Power, X501 Current, X502 I2S, X503 Current, X504 I2C, X505 Current, X506 Current, X507 Current, X508 Current, X509 Motor, X510 Current, X601 DEBUG, X602 Current, X603 Device, X604 UART, X605 GPIO, X606 Current, X607 IO Current, X608 Display, X609 Touch Current, X610 LED Current

Commit message: Update outputs (release)
Other:
- board text added: "0.1855mm"
- board text added: "1.03mm"
- board text added: "Inner1 (GND)"
- board text added: "Inner2"
- board text added: "Plane"
- board text added: "Prepreg"
- board text added: "Total thickness: 1.561mm"
- board text removed: "1.51mm"
- board text removed: "Total thickness: 1.6mm"
